File: Simple/BLT_Preliminary_Avionics_Schematic_Brandon_update_August_8_2021.brd (EAGLE design)
At the start: 118.1 x 61 mm, 12 parts

Commit message: Updated more files
Parts:
- moved 2_CELL_LIPO_BATTERY 5.33 mm to (23.9, 104.9)
- moved U$3 0.51 mm to (61.7, 94.5)
Routing:
- net BAT+: track 47.3 -> 53.2 mm
- net GND: track 6.73 -> 8.61 mm
Changed lines of the file:
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@@
 </autorouter>
 <elements>
-<element name="2_CELL_LIPO_BATTERY" library="SparkFun-Connectors" package="1X02" value="" x="29.21" y="104.902" smashed="yes">
-<attribute name="NAME" x="25.908" y="106.299" size="0.6096" layer="25" font="vector" ratio="20"/>
-<attribute name="VALUE" x="27.94" y="102.87" size="0.6096" layer="27" font="vector" ratio="20"/>
+<element name="2_CELL_LIPO_BATTERY" library="SparkFun-Connectors" package="1X02" value="" x="23.876" y="104.902" smashed="yes">
+<attribute name="NAME" x="20.574" y="106.299" size="0.6096" layer="25" font="vector" ratio="20"/>
+<attribute name="VALUE" x="22.606" y="102.87" size="0.6096" layer="27" font="vector" ratio="20"/>
 </element>
 <element name="BT1" library="Battery_Holder" library_urn="urn:adsk.eagle:library:27510219" package="BAT_3003" package3d_urn="urn:adsk.eagle:package:27510259/2" value="CR2032" x="94.234" y="79.248" smashed="yes" rot="R90">
@@
 <element name="U$1" library="teensy" package="TEENSY41" value="TEENSY41" x="24.13" y="86.36" smashed="yes" rot="R180"/>
 <element name="U$2" library="BLTFootprints" package="MICROBUILDER_1X08_ROUND" value="BMP390" x="88.7476" y="62.5348" smashed="yes" rot="R270"/>
-<element name="U$3" library="BLTFootprints" package="1X04" value="BUCK_CONVERTER3.3V" x="61.214" y="94.488" smashed="yes" rot="R90">
-<attribute name="VOLTAGE" value="3.3V" x="113.284" y="173.228" size="1.778" layer="27" rot="R90" display="off"/>
+<element name="U$3" library="BLTFootprints" package="1X04" value="BUCK_CONVERTER3.3V" x="61.722" y="94.488" smashed="yes" rot="R90">
+<attribute name="VOLTAGE" value="3.3V" x="113.792" y="173.228" size="1.778" layer="27" rot="R90" display="off"/>
 </element>
 <element name="U$4" library="BLTFootprints" package="1X05" value="GT-U7_GPS" x="7.5692" y="73.8632" smashed="yes"/>
@@
 <wire x1="88.74125" y1="71.27875" x2="88.7476" y2="71.2978" width="0.1524" layer="1"/>
 <wire x1="65.405" y1="71.27875" x2="65.33515" y2="71.3105" width="0.1524" layer="1"/>
-<wire x1="61.24575" y1="89.88425" x2="65.24625" y2="85.88375" width="0.254" layer="1"/>
+<wire x1="61.75375" y1="89.37625" x2="65.24625" y2="85.88375" width="0.254" layer="1"/>
 <wire x1="65.24625" y1="71.4375" x2="65.24625" y2="85.88375" width="0.254" layer="1"/>
 <wire x1="65.24625" y1="71.4375" x2="65.33515" y2="71.3105" width="0.1524" layer="1"/>
@@
 <wire x1="7.62" y1="73.914" x2="7.5692" y2="73.8632" width="0.254" layer="1"/>
 <wire x1="17.2085" y1="106.7435" x2="0" y2="106.7435" width="0.254" layer="1"/>
-<wire x1="61.214" y1="94.488" x2="61.214" y2="94.234" width="0.254" layer="1"/>
-<wire x1="61.24575" y1="94.20225" x2="61.214" y2="94.234" width="0.254" layer="1"/>
-<wire x1="61.24575" y1="94.20225" x2="61.24575" y2="89.88425" width="0.254" layer="1"/>
+<wire x1="61.722" y1="94.488" x2="61.75375" y2="94.45625" width="0.254" layer="1"/>
+<wire x1="61.75375" y1="94.45625" x2="61.75375" y2="89.37625" width="0.254" layer="1"/>
 <wire x1="35.2679" y1="68.2244" x2="51.26853125" y2="68.2244" width="0.254" layer="16"/>
 <wire x1="54.0893" y1="69.5833" x2="55.372" y2="70.866" width="0.254" layer="16"/>
@@
 <wire x1="65.33515" y1="71.3105" x2="55.8165" y2="71.3105" width="0.254" layer="1"/>
 <wire x1="55.8165" y1="71.3105" x2="55.372" y2="70.866" width="0.254" layer="1"/>
-<wire x1="61.7190125" y1="103.5812" x2="62.6872" y2="102.6130125" width="0.254" layer="1"/>
-<wire x1="61.214" y1="94.7957875" x2="61.214" y2="94.488" width="0.254" layer="1"/>
-<wire x1="62.6872" y1="96.2689875" x2="61.214" y2="94.7957875" width="0.254" layer="1"/>
-<wire x1="58.0295375" y1="103.5812" x2="61.7190125" y2="103.5812" width="0.254" layer="1"/>
+<wire x1="62.4810125" y1="103.5812" x2="63.1952" y2="102.8670125" width="0.254" layer="1"/>
+<wire x1="61.722" y1="95.3037875" x2="61.722" y2="94.488" width="0.254" layer="1"/>
+<wire x1="63.1952" y1="96.7769875" x2="61.722" y2="95.3037875" width="0.254" layer="1"/>
+<wire x1="58.0295375" y1="103.5812" x2="62.4810125" y2="103.5812" width="0.254" layer="1"/>
 <wire x1="54.9307375" y1="106.68" x2="58.0295375" y2="103.5812" width="0.254" layer="1"/>
-<wire x1="62.6872" y1="102.6130125" x2="62.6872" y2="96.2689875" width="0.254" layer="1"/>
+<wire x1="63.1952" y1="102.8670125" x2="63.1952" y2="96.7769875" width="0.254" layer="1"/>
 <wire x1="17.272" y1="106.68" x2="54.9307375" y2="106.68" width="0.254" layer="1"/>
 <wire x1="0" y1="106.7435" x2="0" y2="101.412" width="0.254" layer="1"/>
@@
 <vertex x="105.174234375" y="47.244" curve="90"/>
 </polygon>
-<wire x1="1.27" y1="104.902" x2="2.728" y2="103.444" width="0.254" layer="1"/>
-<wire x1="2.728" y1="103.444" x2="2.728" y2="100.584" width="0.254" layer="1"/>
-<wire x1="2.728" y1="100.584" x2="2.728" y2="98.872" width="0.254" layer="1"/>
-<wire x1="2.728" y1="98.872" x2="2.794" y2="98.806" width="0.1524" layer="1"/>
-<via x="2.794" y="98.806" extent="1-16" drill="0.35"/>
-<wire x1="88.7476" y1="66.2178" x2="94.244" y2="89.778" width="0" layer="19" extent="1-1"/>
+<wire x1="1.27" y1="104.902" x2="2.728" y2="103.444" width="0.1524" layer="1"/>
+<wire x1="2.728" y1="103.444" x2="2.728" y2="100.584" width="0.1524" layer="1"/>
+<wire x1="94.244" y1="89.778" x2="91.832" y2="89.778" width="0.1524" layer="1"/>
+<wire x1="91.832" y1="89.778" x2="90.932" y2="90.678" width="0.1524" layer="1"/>
+<via x="90.932" y="90.678" extent="1-16" drill="0.35"/>
 </signal>
 <signal name="SCK">
@@
 <wire x1="88.74125" y1="63.65875" x2="88.7476" y2="63.6778" width="0.1524" layer="1"/>
 <wire x1="65.405" y1="63.65875" x2="65.33515" y2="63.6905" width="0.1524" layer="1"/>
-<wire x1="22.70125" y1="78.74" x2="21.59" y2="78.74" width="0.1524" layer="1"/>
-<wire x1="32.0675" y1="69.37375" x2="22.70125" y2="78.74" width="0.1524" layer="1"/>
-<wire x1="35.71875" y1="69.37375" x2="32.0675" y2="69.37375" width="0.1524" layer="1"/>
-<wire x1="36.5125" y1="68.58" x2="35.71875" y2="69.37375" width="0.1524" layer="1"/>
+<wire x1="35.71875" y1="69.37375" x2="36.5125" y2="68.58" width="0.1524" layer="1"/>
 <wire x1="36.5125" y1="61.75375" x2="36.5125" y2="63.02375" width="0.1524" layer="1"/>
 <wire x1="36.5125" y1="63.02375" x2="36.5125" y2="68.58" width="0.1524" layer="1"/>
@@
 <wire x1="24.638" y1="87.63" x2="24.638" y2="81.788" width="0.1524" layer="1"/>
 <wire x1="24.638" y1="87.63" x2="20.574" y2="91.694" width="0.1524" layer="1"/>
+<wire x1="21.59" y1="78.74" x2="30.95625" y2="69.37375" width="0.1524" layer="1"/>
+<wire x1="30.95625" y1="69.37375" x2="35.71875" y2="69.37375" width="0.1524" layer="1"/>
 </signal>
 <signal name="MISO">
@@
 <wire x1="16.51" y1="92.55125" x2="27.14625" y2="92.55125" width="0.1524" layer="1"/>
 <wire x1="15.08125" y1="93.98" x2="16.51" y2="92.55125" width="0.1524" layer="1"/>
-<wire x1="15.08125" y1="95.0595" x2="15.08125" y2="93.98" width="0.1524" layer="1"/>
-<wire x1="6.50875" y1="103.632" x2="15.08125" y2="95.0595" width="0.1524" layer="1"/>
-<wire x1="5.08" y1="103.632" x2="6.50875" y2="103.632" width="0.1524" layer="1"/>
-<wire x1="3.81" y1="104.902" x2="5.08" y2="103.632" width="0.1524" layer="1"/>
+<wire x1="15.08125" y1="94.2975" x2="15.08125" y2="93.98" width="0.1524" layer="1"/>
+<wire x1="13.11275" y1="96.266" x2="15.08125" y2="94.2975" width="0.1524" layer="1"/>
+<wire x1="12.446" y1="96.266" x2="13.11275" y2="96.266" width="0.1524" layer="1"/>
+<wire x1="3.81" y1="104.902" x2="12.446" y2="96.266" width="0.1524" layer="1"/>
 </signal>
 <signal name="CSN">
@@
 <contactref element="U$3" pad="IN+"/>
 <contactref element="U$6" pad="IN+"/>
-<wire x1="54.61" y1="104.902" x2="31.75" y2="104.902" width="0.254" layer="1"/>
-<wire x1="61.214" y1="99.568" x2="59.944" y2="99.568" width="0.254" layer="1"/>
+<wire x1="54.61" y1="104.902" x2="26.416" y2="104.902" width="0.254" layer="1"/>
+<wire x1="61.722" y1="99.568" x2="59.944" y2="99.568" width="0.254" layer="1"/>
 <wire x1="59.944" y1="99.568" x2="59.91225" y2="99.568" width="0.254" layer="1"/>
 <wire x1="59.944" y1="99.568" x2="54.61" y2="104.902" width="0.254" layer="1"/>

Commit message: files updated
Routing:
- net GND: track 8.61 -> 0.00 mm, vias 1 -> 0
- net VBAT: track 113.2 -> 116.3 mm
Other:
- board text added: "Beach Launch Team PCB S2.1"
Changed lines of the file:
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@@
 <wire x1="110.49" y1="103.61395625" x2="110.49" y2="97.536" width="0.0762" layer="20"/>
 <wire x1="-7.62" y1="97.155" x2="-7.62" y2="97.2312" width="0.0254" layer="20"/>
+<text x="8.89" y="99.314" size="1.778" layer="121">Beach Launch Team PCB S2.1</text>
 </plain>
 <attributes>
@@
 <vertex x="105.174234375" y="47.244" curve="90"/>
 </polygon>
-<wire x1="1.27" y1="104.902" x2="2.728" y2="103.444" width="0.1524" layer="1"/>
-<wire x1="2.728" y1="103.444" x2="2.728" y2="100.584" width="0.1524" layer="1"/>
-<wire x1="94.244" y1="89.778" x2="91.832" y2="89.778" width="0.1524" layer="1"/>
-<wire x1="91.832" y1="89.778" x2="90.932" y2="90.678" width="0.1524" layer="1"/>
-<via x="90.932" y="90.678" extent="1-16" drill="0.35"/>
+<wire x1="88.7476" y1="66.2178" x2="94.244" y2="89.778" width="0" layer="19" extent="1-1"/>
+<wire x1="2.728" y1="100.584" x2="1.27" y2="104.902" width="0" layer="19" extent="1-1"/>
 </signal>
 <signal name="SCK">
@@
 <contactref element="BT1" pad="P2"/>
 <wire x1="94.13875" y1="100.33" x2="94.244" y2="100.328" width="0.1524" layer="1"/>
-<wire x1="94.2975" y1="85.4075" x2="94.2975" y2="83.058" width="0.254" layer="1"/>
-<wire x1="94.2975" y1="83.058" x2="94.2975" y2="79.375" width="0.254" layer="1"/>
+<wire x1="94.2975" y1="85.4075" x2="94.2975" y2="83.566" width="0.254" layer="1"/>
+<wire x1="94.2975" y1="83.566" x2="94.2975" y2="79.375" width="0.254" layer="1"/>
 <wire x1="96.52" y1="87.63" x2="94.2975" y2="85.4075" width="0.254" layer="1"/>
 <wire x1="96.52" y1="97.94875" x2="96.52" y2="87.63" width="0.254" layer="1"/>
@@
 <wire x1="23.9404" y1="92.202" x2="31.75" y2="92.202" width="0.254" layer="16"/>
 <via x="31.75" y="92.202" extent="1-16" drill="0.35"/>
-<wire x1="31.75" y1="92.202" x2="55.626" y2="92.202" width="0.254" layer="1"/>
-<wire x1="55.626" y1="92.202" x2="58.42" y2="89.408" width="0.254" layer="1"/>
-<via x="58.42" y="89.408" extent="1-16" drill="0.35"/>
-<wire x1="58.42" y1="89.408" x2="62.992" y2="89.408" width="0.254" layer="16"/>
-<via x="62.992" y="89.408" extent="1-16" drill="0.35"/>
-<wire x1="62.992" y1="89.408" x2="87.9475" y2="89.408" width="0.254" layer="1"/>
-<wire x1="87.9475" y1="89.408" x2="94.2975" y2="83.058" width="0.254" layer="1"/>
+<wire x1="31.75" y1="92.202" x2="55.88" y2="92.202" width="0.254" layer="1"/>
+<wire x1="55.88" y1="92.202" x2="58.928" y2="89.154" width="0.254" layer="1"/>
 <wire x1="9.652" y1="90.678" x2="8.89" y2="91.44" width="0.254" layer="1"/>
 <wire x1="20.574" y1="90.678" x2="9.652" y2="90.678" width="0.254" layer="1"/>
+<wire x1="58.928" y1="89.154" x2="58.928" y2="83.566" width="0.254" layer="1"/>
+<wire x1="58.928" y1="83.566" x2="64.008" y2="83.566" width="0.254" layer="1"/>
+<via x="64.008" y="83.566" extent="1-16" drill="0.35"/>
+<wire x1="64.008" y1="83.566" x2="66.802" y2="83.566" width="0.254" layer="16"/>
+<via x="66.802" y="83.566" extent="1-16" drill="0.35"/>
+<wire x1="66.802" y1="83.566" x2="94.2975" y2="83.566" width="0.254" layer="1"/>
 </signal>
 <signal name="CS1">

Commit message: Updated files
Routing:
- net GND: track 0.00 -> 8.30 mm, vias 0 -> 1
- net SCK: track 120.0 -> 118.6 mm, vias 3 -> 5
Changed lines of the file:
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@@
 <vertex x="105.174234375" y="47.244" curve="90"/>
 </polygon>
-<wire x1="88.7476" y1="66.2178" x2="94.244" y2="89.778" width="0" layer="19" extent="1-1"/>
-<wire x1="2.728" y1="100.584" x2="1.27" y2="104.902" width="0" layer="19" extent="1-1"/>
+<wire x1="94.244" y1="89.778" x2="92.858" y2="88.392" width="0.1524" layer="1"/>
+<wire x1="92.858" y1="88.392" x2="91.44" y2="88.392" width="0.254" layer="1"/>
+<via x="91.44" y="88.392" extent="1-16" drill="0.35"/>
+<wire x1="2.728" y1="100.584" x2="1.27" y2="102.042" width="0.254" layer="1"/>
+<wire x1="1.27" y1="102.042" x2="1.27" y2="104.902" width="0.254" layer="1"/>
 </signal>
 <signal name="SCK">
@@
 <wire x1="88.74125" y1="63.65875" x2="88.7476" y2="63.6778" width="0.1524" layer="1"/>
 <wire x1="65.405" y1="63.65875" x2="65.33515" y2="63.6905" width="0.1524" layer="1"/>
-<wire x1="35.71875" y1="69.37375" x2="36.5125" y2="68.58" width="0.1524" layer="1"/>
-<wire x1="36.5125" y1="61.75375" x2="36.5125" y2="63.02375" width="0.1524" layer="1"/>
-<wire x1="36.5125" y1="63.02375" x2="36.5125" y2="68.58" width="0.1524" layer="1"/>
-<wire x1="35.40125" y1="60.6425" x2="36.5125" y2="61.75375" width="0.1524" layer="1"/>
-<wire x1="35.40125" y1="60.6425" x2="35.2679" y2="60.6044" width="0.1524" layer="1"/>
 <wire x1="7.62" y1="103.632" x2="6.35" y2="104.902" width="0.1524" layer="16"/>
 <wire x1="12.7" y1="94.615" x2="7.62" y2="99.695" width="0.1524" layer="16"/>
@@
 <wire x1="55.08625" y1="63.65875" x2="65.24625" y2="63.65875" width="0.1524" layer="1"/>
 <wire x1="53.49875" y1="62.07125" x2="55.08625" y2="63.65875" width="0.1524" layer="1"/>
-<wire x1="38.735" y1="62.07125" x2="53.49875" y2="62.07125" width="0.1524" layer="1"/>
-<wire x1="37.7825" y1="63.02375" x2="38.735" y2="62.07125" width="0.1524" layer="16"/>
-<wire x1="36.5125" y1="63.02375" x2="37.7825" y2="63.02375" width="0.1524" layer="1"/>
 <wire x1="65.24625" y1="63.65875" x2="65.33515" y2="63.6905" width="0.1524" layer="1"/>
 <via x="12.7" y="94.615" extent="1-16" drill="0.35"/>
-<via x="38.735" y="62.07125" extent="1-16" drill="0.35"/>
-<via x="37.7825" y="63.02375" extent="1-16" drill="0.35"/>
 <wire x1="20.574" y1="91.694" x2="13.716" y2="91.694" width="0.1524" layer="1"/>
 <wire x1="13.716" y1="91.694" x2="12.7" y2="92.71" width="0.1524" layer="1"/>
@@
 <wire x1="24.638" y1="87.63" x2="24.638" y2="81.788" width="0.1524" layer="1"/>
 <wire x1="24.638" y1="87.63" x2="20.574" y2="91.694" width="0.1524" layer="1"/>
-<wire x1="21.59" y1="78.74" x2="30.95625" y2="69.37375" width="0.1524" layer="1"/>
-<wire x1="30.95625" y1="69.37375" x2="35.71875" y2="69.37375" width="0.1524" layer="1"/>
+<wire x1="21.59" y1="78.74" x2="30.988" y2="69.342" width="0.1524" layer="1"/>
+<via x="30.988" y="69.342" extent="1-16" drill="0.35"/>
+<wire x1="30.988" y1="69.342" x2="33.02" y2="67.31" width="0.1524" layer="16"/>
+<via x="33.02" y="67.31" extent="1-16" drill="0.35"/>
+<wire x1="33.02" y1="67.31" x2="33.274" y2="67.056" width="0.254" layer="1"/>
+<wire x1="33.274" y1="67.056" x2="33.274" y2="62.23" width="0.1778" layer="1"/>
+<wire x1="33.274" y1="62.23" x2="34.8996" y2="60.6044" width="0.1524" layer="1"/>
+<wire x1="34.8996" y1="60.6044" x2="35.2679" y2="60.6044" width="0.1524" layer="1"/>
+<wire x1="35.2679" y1="60.6044" x2="37.6555" y2="62.992" width="0.1524" layer="1"/>
+<wire x1="37.6555" y1="62.992" x2="37.846" y2="62.992" width="0.254" layer="1"/>
+<via x="37.846" y="62.992" extent="1-16" drill="0.35"/>
+<wire x1="38.862" y1="62.23" x2="39.02075" y2="62.07125" width="0.1524" layer="1"/>
+<wire x1="53.49875" y1="62.07125" x2="39.02075" y2="62.07125" width="0.1524" layer="1"/>
+<via x="38.862" y="62.23" extent="1-16" drill="0.35"/>
+<wire x1="38.862" y1="62.23" x2="38.608" y2="62.23" width="0.1524" layer="16"/>
+<wire x1="38.608" y1="62.23" x2="37.846" y2="62.992" width="0.1524" layer="16"/>
 </signal>
 <signal name="MISO">

Commit message: Updated files
Parts:
- removed 2_CELL_LIPO_BATTERY: (no value), SparkFun-Connectors:1X02
- added 120: (no value), SparkFun-Resistors:1206
- added CAN_HEADER: (no value), SparkFun-Connectors:1X02_2.54_SCREWTERM
- added LIPO_CONNECTOR: (no value), SparkFun-Connectors:1X02_XTRA_BIG
- added R1: 10k, SparkFun-Resistors:0603
- added U$8: ICM20XXX, BLTFootprints:1X06
- added U1: SN65HVD230, SN65HVD230:SOIC127P599X175-8N
Connections:
- new net CANH: 120.2, CAN_HEADER.P2, U1.7
- new net CANL: 120.1, CAN_HEADER.P1, U1.6
- new net CANRX: U$1.23-A9/CRX1/MCLK1, U1.4
- new net CANTX: U$1.22-A8/CTX1, U1.1
- new net CS3: U$1.16-A2/RX4/SCL1, U$8.CS
- new net ICMINT1: U$1.24-A10/TX6/SCL2, U$8.INT1
- new net ICMINT2: U$1.25-A11/RX6/SDA2, U$8.INT2
- new net SN65RS: R1.2, U1.8
- net 3.3V: now also U$8.VIN, U1.3
- net BAT+: now also LIPO_CONNECTOR.2; no longer 2_CELL_LIPO_BATTERY.2
- net GND: now also LIPO_CONNECTOR.1, R1.1, U$8.GND, U1.2; no longer 2_CELL_LIPO_BATTERY.1
- net MISO: now also U$8.AD0
- net MOSI: now also U$8.SDA
- net SCK: now also U$8.SCL
Routing:
- net ICMINT2: track 0.00 -> 168.5 mm
- net ICMINT1: track 0.00 -> 149.3 mm, vias 0 -> 1
- net CS3: track 0.00 -> 105.2 mm, vias 0 -> 4
- net CANTX: track 0.00 -> 54.4 mm, vias 0 -> 1
- net 3.3V: track 193.7 -> 237.4 mm
- net MISO: track 113.0 -> 153.0 mm
- net CANRX: track 0.00 -> 34.5 mm
- net CANH: track 0.00 -> 33.0 mm, vias 0 -> 1
- net BAT+: track 53.2 -> 25.5 mm
- net SCK: track 118.6 -> 142.2 mm, vias 5 -> 6
- net CANL: track 0.00 -> 21.0 mm
- net MOSI: track 109.9 -> 129.0 mm
- net GND: track 8.30 -> 14.6 mm, vias 1 -> 2
- net SN65RS: track 0.00 -> 2.83 mm
- net TX2: track 30.6 -> 32.3 mm
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Other:
- board size 118.1 x 61 mm -> 138.7 x 61.2 mm

Commit message: Updated files
Routing:
- net VBAT: track 114.7 -> 107.9 mm
Changed lines of the file:
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@@
 <wire x1="131.064" y1="103.61395625" x2="131.064" y2="97.536" width="0.0762" layer="20"/>
 <wire x1="-7.62" y1="97.155" x2="-7.62" y2="97.2312" width="0.0254" layer="20"/>
-<text x="8.89" y="99.314" size="1.778" layer="121">Beach Launch Team PCB S2.1</text>
+<text x="-3.81" y="96.266" size="1.778" layer="121">Beach Launch Team PCB S2.1</text>
 </plain>
 <attributes>
@@
 <contactref element="BT1" pad="P1"/>
 <contactref element="BT1" pad="P2"/>
-<wire x1="94.2975" y1="84.1375" x2="94.2975" y2="79.375" width="0.508" layer="1"/>
-<wire x1="97.79" y1="87.63" x2="94.2975" y2="84.1375" width="0.508" layer="1"/>
-<wire x1="97.79" y1="96.67875" x2="97.79" y2="87.63" width="0.508" layer="1"/>
-<wire x1="94.2975" y1="100.17125" x2="96.218375" y2="98.250375" width="0.508" layer="1"/>
-<wire x1="96.218375" y1="98.250375" x2="97.79" y2="96.67875" width="0.508" layer="1"/>
-<wire x1="94.2975" y1="79.375" x2="94.244" y2="79.228" width="0.508" layer="1"/>
-<wire x1="94.2975" y1="100.17125" x2="94.244" y2="100.328" width="0.508" layer="1"/>
+<wire x1="94.244" y1="79.228" x2="81.27" y2="92.202" width="0.508" layer="1"/>
 <via x="20.32" y="90.932" extent="1-16" drill="0.35"/>
 <wire x1="20.32" y1="90.932" x2="20.45055" y2="90.80145" width="0.508" layer="16"/>
@@
 <wire x1="63.5" y1="92.202" x2="49.784" y2="92.202" width="0.508" layer="16"/>
 <via x="63.5" y="92.202" extent="1-16" drill="0.35"/>
-<wire x1="63.5" y1="92.202" x2="90.17" y2="92.202" width="0.508" layer="1"/>
-<wire x1="90.17" y1="92.202" x2="96.218375" y2="98.250375" width="0.508" layer="1"/>
+<wire x1="63.5" y1="92.202" x2="81.27" y2="92.202" width="0.508" layer="1"/>
+<wire x1="94.244" y1="100.328" x2="86.116" y2="92.2" width="0.508" layer="1"/>
+<wire x1="86.116" y1="92.2" x2="81.29" y2="92.2" width="0.508" layer="1"/>
+<wire x1="81.29" y1="92.2" x2="81.292" y2="92.202" width="0.508" layer="1"/>
+<wire x1="81.292" y1="92.202" x2="81.27" y2="92.202" width="0.508" layer="1"/>
 </signal>
 <signal name="CS1">

Commit message: Updated files
Parts:
- moved U$4 3.34 mm to (10.9, 73.4)
Routing:
- net 3.3V: track 237.4 -> 234.1 mm
Changed lines of the file:
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@@
 <wire x1="125.792121875" y1="46.987553125" x2="131.06178125" y2="51.74911875" width="0" layer="20" curve="90.364639"/>
 <wire x1="131.06178125" y1="51.74911875" x2="131.06178125" y2="97.6124625" width="0" layer="20"/>
-<hole x="-4.318" y="104.648" drill="1"/>
-<hole x="-4.318" y="50.292" drill="1"/>
-<hole x="127.762" y="104.648" drill="1"/>
-<hole x="127.762" y="51.308" drill="1"/>
+<hole x="-3.81" y="104.394" drill="2.5"/>
+<hole x="-3.81" y="50.8" drill="2.5"/>
+<hole x="127.254" y="104.394" drill="2.5"/>
+<hole x="127.254" y="50.8" drill="2.5"/>
 <text x="70.612" y="97.028" size="1.778" layer="121">3.3V</text>
 <text x="72.644" y="84.582" size="1.778" layer="121">5V</text>
@@
 <attribute name="VOLTAGE" value="3.3V" x="113.792" y="173.228" size="1.778" layer="27" rot="R90" display="off"/>
 </element>
-<element name="U$4" library="BLTFootprints" package="1X05" value="GT-U7_GPS" x="7.5692" y="73.8632" smashed="yes"/>
+<element name="U$4" library="BLTFootprints" package="1X05" value="GT-U7_GPS" x="10.8712" y="73.3552" smashed="yes"/>
 <element name="U$5" library="BLTFootprints" package="1X07" value="" x="64.5414" y="72.898" smashed="yes" rot="R270"/>
 <element name="U$6" library="BLTFootprints" package="1X04" value="BUCK_CONVERTER5V" x="61.722" y="79.756" smashed="yes" rot="R90">
@@
 <wire x1="65.24625" y1="71.4375" x2="65.33515" y2="71.3105" width="0.508" layer="1"/>
 <wire x1="19.05" y1="104.902" x2="17.272" y2="106.68" width="0.508" layer="1"/>
-<wire x1="13.17625" y1="68.2625" x2="35.2425" y2="68.2625" width="0.508" layer="1"/>
-<wire x1="7.62" y1="73.81875" x2="13.17625" y2="68.2625" width="0.508" layer="1"/>
+<wire x1="15.3273125" y1="68.2625" x2="35.2425" y2="68.2625" width="0.508" layer="1"/>
 <wire x1="35.2425" y1="68.2625" x2="35.2679" y2="68.2244" width="0.508" layer="1"/>
-<wire x1="7.62" y1="73.81875" x2="7.5692" y2="73.8632" width="0.508" layer="1"/>
+<wire x1="15.3273125" y1="68.2625" x2="10.8712" y2="73.3552" width="0.508" layer="1"/>
 <wire x1="61.722" y1="94.488" x2="62.26175" y2="93.94825" width="0.508" layer="1"/>
 <wire x1="62.26175" y1="93.94825" x2="62.26175" y2="89.37625" width="0.508" layer="1"/>
@@
 <contactref element="U$1" pad="8-TX2/IN1"/>
 <contactref element="U$4" pad="TXD"/>
-<wire x1="15.1892" y1="73.8632" x2="18.034" y2="76.708" width="0.1524" layer="1"/>
+<wire x1="18.4912" y1="73.3552" x2="18.034" y2="73.8124" width="0.1524" layer="1"/>
 <wire x1="18.034" y1="81.28" x2="22.606" y2="85.852" width="0.1524" layer="1"/>
-<wire x1="18.034" y1="76.708" x2="18.034" y2="81.28" width="0.1524" layer="1"/>
+<wire x1="18.034" y1="73.8124" x2="18.034" y2="81.28" width="0.1524" layer="1"/>
 <via x="22.606" y="85.852" extent="1-16" drill="0.35"/>
 <wire x1="22.606" y1="85.852" x2="25.4" y2="88.646" width="0.1524" layer="16"/>
@@
 <via x="22.606" y="88.138" extent="1-16" drill="0.35"/>
 <wire x1="22.606" y1="88.138" x2="14.986" y2="80.518" width="0.1524" layer="1"/>
-<wire x1="14.986" y1="76.2" x2="12.6492" y2="73.8632" width="0.1524" layer="1"/>
-<wire x1="14.986" y1="80.518" x2="14.986" y2="76.2" width="0.1524" layer="1"/>
+<wire x1="14.986" y1="74.3204" x2="15.9512" y2="73.3552" width="0.1524" layer="1"/>
+<wire x1="14.986" y1="80.518" x2="14.986" y2="74.3204" width="0.1524" layer="1"/>
 </signal>
 <signal name="5V">
