File: Simple/BLT_Preliminary_Avionics_Schematic_Brandon_update_August_8_2021.brd (EAGLE design)
At the start: 138.7 x 61.2 mm, 17 parts, among them U1 SN65HVD230

Commit message: updated files
Parts:
- moved 120 1.27 mm to (31.2, 102.4)
Routing:
- net CANH: track 33.0 -> 18.7 mm, vias 1 -> 0
- net GND: track 14.6 -> 12.4 mm, vias 2 -> 3
- net CANL: track 21.0 -> 19.6 mm
- net MOSI: track 129.0 -> 127.7 mm
- net CANTX: track 54.4 -> 55.6 mm, vias 1 -> 0
Changed lines of the file:
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@@
 <attribute name="VALUE" x="22.606" y="99.06" size="0.6096" layer="27" font="vector" ratio="20"/>
 </element>
-<element name="120" library="SparkFun-Resistors" library_urn="urn:adsk.eagle:library:532" package="1206" package3d_urn="urn:adsk.eagle:package:39654/1" value=" " x="31.242" y="103.632" smashed="yes" rot="R270">
-<attribute name="NAME" x="32.385" y="103.632" size="0.6096" layer="25" font="vector" ratio="20" rot="R270" align="bottom-center"/>
-<attribute name="PROD_ID" value=" " x="31.242" y="103.632" size="1.778" layer="27" rot="R270" display="off"/>
-<attribute name="VALUE" x="30.099" y="103.632" size="0.6096" layer="27" font="vector" ratio="20" rot="R270" align="top-center"/>
+<element name="120" library="SparkFun-Resistors" library_urn="urn:adsk.eagle:library:532" package="1206" package3d_urn="urn:adsk.eagle:package:39654/1" value=" " x="31.242" y="102.362" smashed="yes" rot="R270">
+<attribute name="NAME" x="32.385" y="102.362" size="0.6096" layer="25" font="vector" ratio="20" rot="R270" align="bottom-center"/>
+<attribute name="PROD_ID" value=" " x="31.242" y="102.362" size="1.778" layer="27" rot="R270" display="off"/>
+<attribute name="VALUE" x="30.099" y="102.362" size="0.6096" layer="27" font="vector" ratio="20" rot="R270" align="top-center"/>
 </element>
 </elements>
@@
 <wire x1="39.6875" y1="104.4575" x2="39.79" y2="104.648" width="0.1524" layer="1"/>
 <via x="38.608" y="103.378" extent="1-16" drill="0.35"/>
-<wire x1="39.79" y1="104.648" x2="39.79" y2="104.56" width="0.508" layer="1"/>
-<wire x1="39.79" y1="104.56" x2="38.608" y2="103.378" width="0.508" layer="1"/>
-<wire x1="36.138" y1="100.711" x2="37.211" y2="100.711" width="0.508" layer="1"/>
-<wire x1="38.608" y1="102.108" x2="38.608" y2="103.378" width="0.508" layer="1"/>
-<wire x1="37.211" y1="100.711" x2="38.608" y2="102.108" width="0.508" layer="1"/>
+<wire x1="39.116" y1="104.648" x2="38.608" y2="104.14" width="0.508" layer="1"/>
+<wire x1="38.608" y1="104.14" x2="38.608" y2="103.378" width="0.508" layer="1"/>
+<wire x1="39.79" y1="104.648" x2="39.116" y2="104.648" width="0.508" layer="1"/>
+<wire x1="37.719" y1="100.711" x2="37.846" y2="100.838" width="0.508" layer="1"/>
+<wire x1="36.138" y1="100.711" x2="37.719" y2="100.711" width="0.508" layer="1"/>
+<via x="37.846" y="100.838" extent="1-16" drill="0.35"/>
 </signal>
 <signal name="SCK">
@@
 <wire x1="29.7815" y1="95.09125" x2="28.8925" y2="95.09125" width="0.1524" layer="1"/>
 <wire x1="29.7815" y1="95.09125" x2="30.38475" y2="94.488" width="0.1524" layer="1"/>
-<wire x1="39.84625" y1="79.85125" x2="44.7675" y2="79.85125" width="0.1524" layer="1"/>
-<wire x1="45.87875" y1="78.74" x2="44.7675" y2="79.85125" width="0.1524" layer="1"/>
-<wire x1="45.87875" y1="78.74" x2="45.87875" y2="65.24625" width="0.1524" layer="1"/>
+<wire x1="45.87875" y1="65.24625" x2="45.87875" y2="75.184" width="0.1524" layer="1"/>
 <wire x1="48.41875" y1="62.70625" x2="45.87875" y2="65.24625" width="0.1524" layer="1"/>
 <wire x1="53.0225" y1="58.1025" x2="48.41875" y2="62.70625" width="0.1524" layer="16"/>
@@
 <wire x1="29.718" y1="92.456" x2="29.718" y2="89.9795" width="0.1524" layer="1"/>
 <wire x1="30.38475" y1="94.488" x2="30.38475" y2="93.12275" width="0.1524" layer="1"/>
-<wire x1="29.718" y1="89.9795" x2="39.84625" y2="79.85125" width="0.1524" layer="1"/>
+<wire x1="39.84625" y1="79.85125" x2="29.718" y2="89.9795" width="0.1524" layer="1"/>
+<wire x1="45.87875" y1="75.184" x2="43.18" y2="77.88275" width="0.1524" layer="1"/>
+<wire x1="43.18" y1="77.88275" x2="43.18" y2="79.248" width="0.1524" layer="1"/>
+<wire x1="43.18" y1="79.248" x2="42.57675" y2="79.85125" width="0.1524" layer="1"/>
+<wire x1="42.57675" y1="79.85125" x2="39.84625" y2="79.85125" width="0.1524" layer="1"/>
 </signal>
 <signal name="CS">
@@
 <contactref element="120" pad="2"/>
 <contactref element="CAN_HEADER" pad="P2"/>
-<wire x1="24.13" y1="101.9175" x2="31.115" y2="101.9175" width="0.1524" layer="1"/>
-<wire x1="24.13" y1="102.87" x2="24.13" y2="101.9175" width="0.1524" layer="1"/>
-<wire x1="31.115" y1="101.9175" x2="31.242" y2="102.232" width="0.1524" layer="1"/>
-<wire x1="24.13" y1="102.87" x2="23.876" y2="103.124" width="0.1524" layer="1"/>
-<wire x1="42.545" y1="100.6475" x2="41.275" y2="100.6475" width="0.1524" layer="1"/>
-<wire x1="42.545" y1="99.06" x2="42.545" y2="100.6475" width="0.1524" layer="1"/>
-<wire x1="42.2275" y1="98.7425" x2="42.545" y2="99.06" width="0.1524" layer="1"/>
-<wire x1="27.813" y1="98.7425" x2="42.2275" y2="98.7425" width="0.1524" layer="1"/>
-<wire x1="27.6225" y1="98.552" x2="27.813" y2="98.7425" width="0.1524" layer="1"/>
-<wire x1="23.7109" y1="102.4636" x2="27.6225" y2="98.552" width="0.1524" layer="16"/>
-<wire x1="41.275" y1="100.6475" x2="41.078" y2="100.711" width="0.1524" layer="1"/>
-<wire x1="23.7109" y1="102.4636" x2="23.876" y2="103.124" width="0.1524" layer="16"/>
-<via x="27.6225" y="98.552" extent="1-16" drill="0.35"/>
+<wire x1="26.0985" y1="100.9015" x2="23.876" y2="103.124" width="0.1524" layer="1"/>
+<wire x1="41.078" y1="100.711" x2="38.57715" y2="100.711" width="0.1524" layer="1"/>
+<wire x1="38.57715" y1="100.711" x2="38.04855" y2="100.1824" width="0.1524" layer="1"/>
+<wire x1="31.242" y1="100.962" x2="31.1815" y2="100.9015" width="0.1524" layer="1"/>
+<wire x1="31.1815" y1="100.9015" x2="26.0985" y2="100.9015" width="0.1524" layer="1"/>
+<wire x1="38.04855" y1="100.1824" x2="31.9006" y2="100.1824" width="0.1524" layer="1"/>
+<wire x1="31.9006" y1="100.1824" x2="31.1815" y2="100.9015" width="0.1524" layer="1"/>
 </signal>
 <signal name="CANL">
@@
 <contactref element="120" pad="1"/>
 <contactref element="CAN_HEADER" pad="P1"/>
-<wire x1="26.67" y1="104.775" x2="31.115" y2="104.775" width="0.1524" layer="1"/>
-<wire x1="26.67" y1="103.1875" x2="26.67" y2="104.775" width="0.1524" layer="1"/>
-<wire x1="31.115" y1="104.775" x2="31.242" y2="105.032" width="0.1524" layer="1"/>
-<wire x1="26.67" y1="103.1875" x2="26.416" y2="103.124" width="0.1524" layer="1"/>
-<wire x1="37.465" y1="99.695" x2="40.9575" y2="99.695" width="0.1524" layer="1"/>
-<wire x1="37.1475" y1="100.0125" x2="37.465" y2="99.695" width="0.1524" layer="1"/>
-<wire x1="32.385" y1="100.0125" x2="37.1475" y2="100.0125" width="0.1524" layer="1"/>
-<wire x1="32.385" y1="103.8225" x2="32.385" y2="100.0125" width="0.1524" layer="1"/>
-<wire x1="31.4325" y1="104.775" x2="32.385" y2="103.8225" width="0.1524" layer="1"/>
-<wire x1="40.9575" y1="99.695" x2="41.078" y2="99.441" width="0.1524" layer="1"/>
-<wire x1="31.4325" y1="104.775" x2="31.242" y2="105.032" width="0.1524" layer="1"/>
+<wire x1="30.988" y1="103.508" x2="31.242" y2="103.762" width="0.1524" layer="1"/>
+<wire x1="30.988" y1="103.508" x2="30.73548125" y2="102.997" width="0.1524" layer="1"/>
+<wire x1="31.253340625" y1="103.777303125" x2="31.242" y2="103.762" width="0.1524" layer="1"/>
+<wire x1="42.2916" y1="100.36024375" x2="42.2916" y2="101.06175625" width="0.1524" layer="1"/>
+<wire x1="42.2916" y1="100.36024375" x2="41.37235625" y2="99.441" width="0.1524" layer="1"/>
+<wire x1="41.078" y1="99.441" x2="41.37235625" y2="99.441" width="0.1524" layer="1"/>
+<wire x1="33.57824375" y1="101.4524" x2="31.253340625" y2="103.777303125" width="0.1524" layer="1"/>
+<wire x1="42.2916" y1="101.06175625" x2="41.90095625" y2="101.4524" width="0.1524" layer="1"/>
+<wire x1="41.90095625" y1="101.4524" x2="33.57824375" y2="101.4524" width="0.1524" layer="1"/>
+<wire x1="30.604" y1="103.124" x2="26.416" y2="103.124" width="0.1524" layer="1"/>
+<wire x1="30.604" y1="103.124" x2="30.73548125" y2="102.997" width="0" layer="19" extent="1-1"/>
 </signal>
 <signal name="CANTX">
 <contactref element="U1" pad="1"/>
 <contactref element="U$1" pad="22-A8/CTX1"/>
-<wire x1="39.0525" y1="105.41" x2="36.138" y2="102.4955" width="0.1524" layer="1"/>
-<wire x1="51.1175" y1="101.6" x2="51.1175" y2="104.14" width="0.1524" layer="1"/>
-<wire x1="53.34" y1="77.597" x2="53.34" y2="99.3775" width="0.1524" layer="1"/>
+<wire x1="38.2905" y1="105.918" x2="36.138" y2="103.7655" width="0.1524" layer="1"/>
+<wire x1="53.34" y1="77.597" x2="53.34" y2="94.742" width="0.1524" layer="1"/>
 <wire x1="52.8955" y1="77.1525" x2="53.34" y2="77.597" width="0.1524" layer="1"/>
-<wire x1="46.6725" y1="77.1525" x2="52.8955" y2="77.1525" width="0.1524" layer="1"/>
-<wire x1="45.72" y1="78.105" x2="46.6725" y2="77.1525" width="0.1524" layer="16"/>
-<wire x1="45.4025" y1="78.105" x2="45.72" y2="78.105" width="0.1524" layer="16"/>
-<wire x1="44.7675" y1="78.74" x2="45.4025" y2="78.105" width="0.1524" layer="16"/>
-<wire x1="44.45" y1="78.74" x2="44.7675" y2="78.74" width="0.1524" layer="16"/>
-<wire x1="36.138" y1="102.4955" x2="36.138" y2="101.981" width="0.1524" layer="1"/>
-<via x="46.6725" y="77.1525" extent="1-16" drill="0.35"/>
-<wire x1="53.34" y1="99.3775" x2="51.1175" y2="101.6" width="0.1524" layer="1"/>
-<wire x1="51.1175" y1="104.14" x2="49.8475" y2="105.41" width="0.1524" layer="1"/>
-<wire x1="39.0525" y1="105.41" x2="49.8475" y2="105.41" width="0.1524" layer="1"/>
+<wire x1="46.0375" y1="77.1525" x2="52.8955" y2="77.1525" width="0.1524" layer="1"/>
+<wire x1="36.138" y1="103.7655" x2="36.138" y2="101.981" width="0.1524" layer="1"/>
+<wire x1="38.2905" y1="105.918" x2="42.672" y2="105.918" width="0.1524" layer="1"/>
+<wire x1="42.672" y1="105.918" x2="43.9674" y2="104.6226" width="0.1524" layer="1"/>
+<wire x1="43.9674" y1="104.6226" x2="43.9674" y2="97.4668375" width="0.1524" layer="1"/>
+<wire x1="45.4222375" y1="96.012" x2="43.9674" y2="97.4668375" width="0.1524" layer="1"/>
+<wire x1="53.34" y1="94.742" x2="52.07" y2="96.012" width="0.1524" layer="1"/>
+<wire x1="52.07" y1="96.012" x2="45.4222375" y2="96.012" width="0.1524" layer="1"/>
+<wire x1="46.0375" y1="77.1525" x2="44.45" y2="78.74" width="0.1524" layer="1"/>
 </signal>
 <signal name="CANRX">

Commit message: Updated files
Parts:
- moved BT1 10.4 mm to (104.6, 79.0)
- moved U$3 10.4 mm to (72.1, 94.2)
- moved U$6 10.4 mm to (72.1, 79.5)
Routing:
- net 3.3V: track 234.1 -> 249.9 mm
- net VBAT: track 107.9 -> 118.5 mm, vias 4 -> 6
- net BAT+: track 25.5 -> 36.0 mm
- net 5V: track 7.53 -> 17.8 mm
- net CS3: track 105.2 -> 114.4 mm, vias 4 -> 2
