File: Simple/BLT_Preliminary_Avionics_Schematic_Brandon_update_August_8_2021.brd (EAGLE design)
At the start: 138.7 x 61.2 mm, 17 parts, among them U1 SN65HVD230

Commit message: updated files
Routing:
- net 3.3V: track 249.9 -> 240.7 mm
- net ICMINT2: track 168.5 -> 170.2 mm
- net CS3: track 114.4 -> 113.7 mm

Commit message: Updated files
Parts:
- removed CAN_HEADER: (no value), SparkFun-Connectors:1X02_2.54_SCREWTERM
- added CAN_CONNECTOR: (no value), SparkFun-Connectors:1X03
- added LIPO_CONNECTOR_2: (no value), SparkFun-Connectors:1X02
- moved C6 17.4 mm to (19.1, 102.4)
- moved 120 1.78 mm to (33.0, 102.4), turned to 90 degrees
Connections:
- net BAT+: now also LIPO_CONNECTOR_2.2
- net CANH: now also CAN_CONNECTOR.3; no longer CAN_HEADER.P2
- net CANL: now also CAN_CONNECTOR.2; no longer CAN_HEADER.P1
- net GND: now also CAN_CONNECTOR.1, LIPO_CONNECTOR_2.1
Routing:
- net 3.3V: track 240.7 -> 217.7 mm
- net CANH: track 18.7 -> 14.0 mm
- net GND: track 12.2 -> 8.13 mm, vias 3 -> 4
- net CANL: track 19.7 -> 17.2 mm
- net BAT+: track 36.0 -> 38.2 mm
- net CANTX: track 55.6 -> 53.9 mm
- net CSN: track 15.1 -> 16.6 mm
- net CANRX: track 34.5 -> 33.5 mm
- net MOSI: track 127.7 -> 128.3 mm
Other:
- board text added: "BAT+"
- board text added: "CANH"
- board text added: "CANL"
- board text added: "CE"
- board text added: "CSN"
- board text added: "GND"
- board text added: "MISO"
- board text added: "MOSI"
- board text added: "NRF24L01_A"
- board text added: "PPS"
- board text added: "RXD"
- board text added: "SCK"
- board text added: "TXD"
- board text added: "VCC"

Commit message: updated mor files
Parts:
- moved C6 0.57 mm to (19.6, 102.1)
Changed lines of the file:
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@@
 <attribute name="VALUE" x="114.958" y="89.894" size="1" layer="27" rot="R90" align="center"/>
 </element>
-<element name="C6" library="microbuilder" package="0805" value="47uF" x="19.05" y="102.362" smashed="yes">
-<attribute name="NAME" x="21.082" y="102.235" size="0.8128" layer="25" ratio="18"/>
-<attribute name="VALUE" x="21.082" y="101.6" size="0.4064" layer="27" ratio="10"/>
+<element name="C6" library="microbuilder" package="0805" value="47uF" x="19.558" y="102.108" smashed="yes">
+<attribute name="NAME" x="21.59" y="101.981" size="0.8128" layer="25" ratio="18"/>
+<attribute name="VALUE" x="21.59" y="101.346" size="0.4064" layer="27" ratio="10"/>
 </element>
 <element name="NRF24L01_A" library="SparkFun-Connectors" library_urn="urn:adsk.eagle:library:513" package="1X04" package3d_urn="urn:adsk.eagle:package:38085/1" value="" x="1.27" y="104.902" smashed="yes">
@@
 <wire x1="88.5627875" y1="71.2730625" x2="74.64425" y2="85.1916" width="0.508" layer="1"/>
 <wire x1="19.05" y1="104.902" x2="20.828" y2="106.68" width="0.508" layer="1"/>
-<wire x1="19.05" y1="104.902" x2="18.1" y2="103.952" width="0.508" layer="1"/>
-<wire x1="18.1" y1="103.952" x2="18.1" y2="102.362" width="0.508" layer="1"/>
+<wire x1="19.05" y1="104.902" x2="18.608" y2="104.46" width="0.508" layer="1"/>
+<wire x1="18.608" y1="104.46" x2="18.608" y2="102.108" width="0.508" layer="1"/>
 <wire x1="22.098" y1="105.664" x2="23.114" y2="106.68" width="0.508" layer="1"/>
 </signal>
@@
 <contactref element="LIPO_CONNECTOR_2" pad="1"/>
 <contactref element="CAN_CONNECTOR" pad="1"/>
-<wire x1="20.066" y1="100.838" x2="20" y2="100.904" width="0.508" layer="1"/>
-<wire x1="20" y1="102.362" x2="20" y2="100.904" width="0.508" layer="1"/>
-<via x="20.066" y="100.838" extent="1-16" drill="0.35"/>
+<wire x1="20.508" y1="102.108" x2="20.508" y2="100.904" width="0.508" layer="1"/>
+<wire x1="20.574" y1="100.838" x2="20.508" y2="100.904" width="0.508" layer="1"/>
+<via x="20.574" y="100.838" extent="1-16" drill="0.35"/>
 </signal>
 <signal name="SCK">

Commit message: Updated files
Parts:
- added RECOVERY_HEADER: (no value), SparkFun-Connectors:1X04
Connections:
- new net RCV1: RECOVERY_HEADER.3, U$1.26-A12/MOSI1
- new net RCV2: RECOVERY_HEADER.4, U$1.27-A13/SCK1
- net BAT+: now also RECOVERY_HEADER.1
- net GND: now also RECOVERY_HEADER.2
Routing:
- net RCV2: track 0.00 -> 101.9 mm, vias 0 -> 3
- net RCV1: track 0.00 -> 101.6 mm, vias 0 -> 3
- net BAT+: track 38.2 -> 63.7 mm, vias 0 -> 1
- net 3.3V: track 217.7 -> 215.5 mm
Other:
- board size 138.7 x 61.2 mm -> 138.9 x 61.2 mm
