File: Simple/BLT_Preliminary_Avionics_Schematic_Brandon_update_August_8_2021.sch (EAGLE design)
At the start: 12 parts

Commit message: Updated files
Parts:
- removed 2_CELL_LIPO_BATTERY: (no value), SparkFun-Connectors:CONN_02
- added 120: (no value), SparkFun-Resistors:RESISTOR1206
- added CAN_HEADER: (no value), SparkFun-Connectors:CONN_022.54MM_SCREWTERM
- added LIPO_CONNECTOR: (no value), SparkFun-Connectors:CONN_02PTH4
- added R1: 10k, SparkFun-Resistors:10KOHM-0603-1/10W-1%
- added U$8: ICM20XXX, BLTFootprints:ICM20XXX
- added U1: SN65HVD230, SN65HVD230:SN65HVD230
Connections:
- new net CANH: 120.2, CAN_HEADER.2, U1.CANH
- new net CANL: 120.1, CAN_HEADER.1, U1.CANL
- new net CANRX: U$1.23-A9/CRX1/MCLK1, U1.R
- new net CANTX: U$1.22-A8/CTX1, U1.D
- new net CS3: U$1.16-A2/RX4/SCL1, U$8.CS
- new net ICMINT1: U$1.24-A10/TX6/SCL2, U$8.INT1
- new net ICMINT2: U$1.25-A11/RX6/SDA2, U$8.INT2
- new net SN65RS: R1.2, U1.RS
- net 3.3V: now also U$8.VCC, U1.VCC
- net BAT+: now also LIPO_CONNECTOR.2; no longer 2_CELL_LIPO_BATTERY.2
- net GND: now also LIPO_CONNECTOR.1, R1.1, U$8.GND, U1.GND; no longer 2_CELL_LIPO_BATTERY.1
- net MISO: now also U$8.AD0
- net MOSI: now also U$8.SDA
- net SCK: now also U$8.SCL

Commit message: Updated files
Parts:
- removed CAN_HEADER: (no value), SparkFun-Connectors:CONN_022.54MM_SCREWTERM
- added CAN_CONNECTOR: (no value), SparkFun-Connectors:CONN_03
- added LIPO_CONNECTOR_2: (no value), SparkFun-Connectors:CONN_02
Connections:
- net BAT+: now also LIPO_CONNECTOR_2.2
- net CANH: now also CAN_CONNECTOR.3; no longer CAN_HEADER.2
- net CANL: now also CAN_CONNECTOR.2; no longer CAN_HEADER.1
- net GND: now also CAN_CONNECTOR.1, LIPO_CONNECTOR_2.1
Changed lines of the file:
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@@
 <part name="U1" library="SN65HVD230" deviceset="SN65HVD230" device=""/>
 <part name="R1" library="SparkFun-Resistors" library_urn="urn:adsk.eagle:library:532" deviceset="10KOHM" device="-0603-1/10W-1%" package3d_urn="urn:adsk.eagle:package:39650/1" value="10k"/>
-<part name="CAN_HEADER" library="SparkFun-Connectors" library_urn="urn:adsk.eagle:library:513" deviceset="CONN_02" device="2.54MM_SCREWTERM" package3d_urn="urn:adsk.eagle:package:38059/1"/>
 <part name="120" library="SparkFun-Resistors" library_urn="urn:adsk.eagle:library:532" deviceset="RESISTOR" device="1206" package3d_urn="urn:adsk.eagle:package:39654/1" value=" "/>
+<part name="LIPO_CONNECTOR_2" library="SparkFun-Connectors" library_urn="urn:adsk.eagle:library:513" deviceset="CONN_02" device="" package3d_urn="urn:adsk.eagle:package:38039/1"/>
+<part name="CAN_CONNECTOR" library="SparkFun-Connectors" library_urn="urn:adsk.eagle:library:513" deviceset="CONN_03" device="" package3d_urn="urn:adsk.eagle:package:38063/1"/>
 </parts>
 <sheets>
@@
 <attribute name="VALUE" x="175.26" y="13.716" size="1.778" layer="96" font="vector" align="top-center"/>
 </instance>
-<instance part="CAN_HEADER" gate="G$1" x="165.1" y="-5.08" smashed="yes">
-<attribute name="VALUE" x="162.56" y="-9.906" size="1.778" layer="96" font="vector"/>
-<attribute name="NAME" x="154.94" y="0.508" size="1.778" layer="95" font="vector"/>
-</instance>
 <instance part="120" gate="G$1" x="177.8" y="5.08" smashed="yes" rot="R180">
 <attribute name="NAME" x="177.8" y="3.556" size="1.778" layer="95" font="vector" rot="R180" align="bottom-center"/>
 <attribute name="VALUE" x="177.8" y="6.604" size="1.778" layer="96" font="vector" rot="R180" align="top-center"/>
+</instance>
+<instance part="LIPO_CONNECTOR_2" gate="G$1" x="152.4" y="96.52" smashed="yes">
+<attribute name="VALUE" x="149.86" y="91.694" size="1.778" layer="96" font="vector"/>
+<attribute name="NAME" x="149.86" y="102.108" size="1.778" layer="95" font="vector"/>
+</instance>
+<instance part="CAN_CONNECTOR" gate="J$1" x="165.1" y="-17.78" smashed="yes">
+<attribute name="VALUE" x="162.56" y="-25.146" size="1.778" layer="96" font="vector"/>
+<attribute name="NAME" x="162.56" y="-12.192" size="1.778" layer="95" font="vector"/>
 </instance>
 </instances>
@@
 <label x="167.64" y="22.86" size="1.778" layer="95"/>
 </segment>
+<segment>
+<pinref part="LIPO_CONNECTOR_2" gate="G$1" pin="1"/>
+<wire x1="160.02" y1="96.52" x2="162.56" y2="96.52" width="0.1524" layer="91"/>
+<label x="162.56" y="96.52" size="1.778" layer="95"/>
+</segment>
+<segment>
+<pinref part="CAN_CONNECTOR" gate="J$1" pin="1"/>
+<wire x1="172.72" y1="-20.32" x2="177.8" y2="-20.32" width="0.1524" layer="91"/>
+<label x="177.8" y="-20.32" size="1.778" layer="95"/>
+</segment>
 </net>
 <net name="SCK" class="0">
@@
 <label x="162.56" y="114.3" size="1.778" layer="95"/>
 </segment>
+<segment>
+<pinref part="LIPO_CONNECTOR_2" gate="G$1" pin="2"/>
+<wire x1="160.02" y1="99.06" x2="162.56" y2="99.06" width="0.1524" layer="91"/>
+<label x="162.56" y="99.06" size="1.778" layer="95"/>
+</segment>
 </net>
 <net name="VBAT" class="0">
@@
 <pinref part="120" gate="G$1" pin="2"/>
 <wire x1="172.72" y1="10.16" x2="172.72" y2="5.08" width="0.1524" layer="91"/>
-<pinref part="CAN_HEADER" gate="G$1" pin="2"/>
-<wire x1="172.72" y1="5.08" x2="172.72" y2="-2.54" width="0.1524" layer="91"/>
-<junction x="172.72" y="5.08"/>
 <label x="177.8" y="10.16" size="1.778" layer="95"/>
+</segment>
+<segment>
+<pinref part="CAN_CONNECTOR" gate="J$1" pin="3"/>
+<wire x1="172.72" y1="-15.24" x2="177.8" y2="-15.24" width="0.1524" layer="91"/>
+<label x="177.8" y="-15.24" size="1.778" layer="95"/>
 </segment>
 </net>
@@
 <wire x1="185.42" y1="7.62" x2="182.88" y2="7.62" width="0.1524" layer="91"/>
 <wire x1="182.88" y1="7.62" x2="182.88" y2="5.08" width="0.1524" layer="91"/>
-<wire x1="182.88" y1="5.08" x2="182.88" y2="-5.08" width="0.1524" layer="91"/>
-<junction x="182.88" y="5.08"/>
-<pinref part="CAN_HEADER" gate="G$1" pin="1"/>
-<wire x1="182.88" y1="-5.08" x2="172.72" y2="-5.08" width="0.1524" layer="91"/>
-<label x="172.72" y="-7.62" size="1.778" layer="95"/>
-</segment>
-</net>
+<label x="182.88" y="2.54" size="1.778" layer="95"/>
+</segment>
+<segment>
+<pinref part="CAN_CONNECTOR" gate="J$1" pin="2"/>
+<wire x1="172.72" y1="-17.78" x2="177.8" y2="-17.78" width="0.1524" layer="91"/>
+<label x="177.8" y="-17.78" size="1.778" layer="95"/>
+</segment>
+</net>

Commit message: Updated files
Parts:
- added RECOVERY_HEADER: (no value), SparkFun-Connectors:CONN_04
Connections:
- new net RCV1: RECOVERY_HEADER.3, U$1.26-A12/MOSI1
- new net RCV2: RECOVERY_HEADER.4, U$1.27-A13/SCK1
- net BAT+: now also RECOVERY_HEADER.1
- net GND: now also RECOVERY_HEADER.2
Changed lines of the file:
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@@
 <part name="LIPO_CONNECTOR_2" library="SparkFun-Connectors" library_urn="urn:adsk.eagle:library:513" deviceset="CONN_02" device="" package3d_urn="urn:adsk.eagle:package:38039/1"/>
 <part name="CAN_CONNECTOR" library="SparkFun-Connectors" library_urn="urn:adsk.eagle:library:513" deviceset="CONN_03" device="" package3d_urn="urn:adsk.eagle:package:38063/1"/>
+<part name="RECOVERY_HEADER" library="SparkFun-Connectors" library_urn="urn:adsk.eagle:library:513" deviceset="CONN_04" device="" package3d_urn="urn:adsk.eagle:package:38085/1"/>
 </parts>
 <sheets>
@@
 <attribute name="VALUE" x="162.56" y="-25.146" size="1.778" layer="96" font="vector"/>
 <attribute name="NAME" x="162.56" y="-12.192" size="1.778" layer="95" font="vector"/>
+</instance>
+<instance part="RECOVERY_HEADER" gate="G$1" x="88.9" y="99.06" smashed="yes" rot="R180">
+<attribute name="VALUE" x="93.98" y="106.426" size="1.778" layer="96" font="vector" rot="R180"/>
+<attribute name="NAME" x="93.98" y="90.932" size="1.778" layer="95" font="vector" rot="R180"/>
 </instance>
 </instances>
@@
 <label x="177.8" y="-20.32" size="1.778" layer="95"/>
 </segment>
+<segment>
+<pinref part="RECOVERY_HEADER" gate="G$1" pin="2"/>
+<wire x1="83.82" y1="99.06" x2="76.2" y2="99.06" width="0.1524" layer="91"/>
+<label x="76.2" y="99.06" size="1.778" layer="95"/>
+</segment>
 </net>
 <net name="SCK" class="0">
@@
 <wire x1="160.02" y1="99.06" x2="162.56" y2="99.06" width="0.1524" layer="91"/>
 <label x="162.56" y="99.06" size="1.778" layer="95"/>
+</segment>
+<segment>
+<pinref part="RECOVERY_HEADER" gate="G$1" pin="1"/>
+<wire x1="83.82" y1="101.6" x2="76.2" y2="101.6" width="0.1524" layer="91"/>
+<label x="76.2" y="101.6" size="1.778" layer="95"/>
 </segment>
 </net>
@@
 </segment>
 </net>
+<net name="RCV1" class="0">
+<segment>
+<pinref part="U$1" gate="G$1" pin="26-A12/MOSI1"/>
+<wire x1="22.86" y1="45.72" x2="20.32" y2="45.72" width="0.1524" layer="91"/>
+<label x="15.24" y="45.72" size="1.778" layer="95"/>
+</segment>
+<segment>
+<pinref part="RECOVERY_HEADER" gate="G$1" pin="3"/>
+<wire x1="83.82" y1="96.52" x2="76.2" y2="96.52" width="0.1524" layer="91"/>
+<label x="76.2" y="96.52" size="1.778" layer="95"/>
+</segment>
+</net>
+<net name="RCV2" class="0">
+<segment>
+<pinref part="U$1" gate="G$1" pin="27-A13/SCK1"/>
+<wire x1="22.86" y1="43.18" x2="20.32" y2="43.18" width="0.1524" layer="91"/>
+<label x="15.24" y="43.18" size="1.778" layer="95"/>
+</segment>
+<segment>
+<pinref part="RECOVERY_HEADER" gate="G$1" pin="4"/>
+<wire x1="83.82" y1="93.98" x2="76.2" y2="93.98" width="0.1524" layer="91"/>
+<label x="76.2" y="93.98" size="1.778" layer="95"/>
+</segment>
+</net>
