File: BLT_Preliminary_Avionics_Schematic_Brandon_update_August_8_2021.brd (EAGLE design)
At the start: 144.8 x 55.5 mm, 25 parts, among them Y1 32.768kHz

Commit message: /
Parts:
- added C6: 470nF, SparkFun-Capacitors:0402
- added R2, R4: 4.7K, OPL_Resistor:R0402
- added U$8, U$9: 10K, OPL_Resistor:R0402
- R1: value (none) -> 4.7K; device microbuilder:0603 -> OPL_Resistor:R0402
- R3: value (none) -> 4.7K; device microbuilder:RESPACK_4X0603 -> OPL_Resistor:R0402
- moved R1 73.1 mm to (-2.54, -6.35)
- moved R3 71.6 mm to (-12.7, -6.35)
Connections:
- new net BMPINT: U$1.20-A6/TX5/LRCLK1, U$3.7
- new net ICMINT1: U$1.16-A2/RX4/SCL1, U$2.12
- new net ICMINT2: U$1.17-A3/TX4/SDA1, U$2.19
- new net N$7: U$8.2, U2.14
- new net N$8: U$9.2, U2.4
- net 3.3V: now also C6.2, R2.2, R3.1, R4.1, U$8.1, U$9.1; no longer R3.5, R3.6, R3.7, R3.8
- net GND: now also C6.1
- net N$3: now also R3.2, U2.16; no longer R3.3, U2.14
- net N$5: no longer R3.4
- net N$6: now also R4.2, U2.15; no longer R1.1, U2.11
- net SCL: now also R2.1; no longer R3.2
- net SDA: now also R1.1; no longer R3.1
Routing:
- net N$3: track 22.5 -> 0.00 mm
- net N$6: track 4.63 -> 0.00 mm
- net 3.3V: track 192.6 -> 189.3 mm

Commit message: Updated files
Parts:
- added U$10: 10K, OPL_Resistor:R0402
- C6: value 470nF -> 47uF; device SparkFun-Capacitors:0402 -> microbuilder:0805
- moved C6 101.4 mm to (41.9, 49.5)
- moved R4 92.8 mm to (62.2, 40.6), turned to 90 degrees
- moved U$9 88.4 mm to (34.3, 44.5)
- moved R3 85.3 mm to (55.9, 44.5), turned to 90 degrees
- moved R2 84.6 mm to (55.9, 49.5), turned to 180 degrees
- moved U$8 83.6 mm to (39.4, 35.6), turned to 90 degrees
- moved R1 77.3 mm to (50.8, 49.5), turned to 180 degrees
- moved C4 62.9 mm to (29.2, 49.5)
- moved C5 58.5 mm to (30.5, 47.0)
- moved Y1 53.1 mm to (34.3, 49.5), turned to 270 degrees
- moved C3 46.0 mm to (38.1, 40.6)
- moved U$3 40.7 mm to (64.8, 34.3)
- moved C2 35.8 mm to (48.3, 38.1), turned to 180 degrees
- moved U2 29.6 mm to (45.7, 44.5)
- moved BT1 24.4 mm to (5.08, 39.4)
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Connections:
- net 3.3V: now also C6.1, U$10.1; no longer C6.2
- net GND: now also C6.2; no longer C6.1
- net N$5: now also U$10.2
Routing:
- net BMPINT: track 0.00 -> 55.1 mm
- net MOSI: track 74.1 -> 117.5 mm, vias 0 -> 2
- net ICMINT1: track 0.00 -> 29.7 mm
- net CSN: track 20.9 -> 48.7 mm
- net ICMINT2: track 0.00 -> 25.0 mm, vias 0 -> 1
- net CS3: track 41.7 -> 17.2 mm, vias 5 -> 1
- net SCL: track 66.7 -> 43.3 mm, vias 6 -> 2
- net CE: track 23.5 -> 45.3 mm
- net GND: track 177.3 -> 198.5 mm, vias 7 -> 10
- net SDA: track 65.4 -> 47.9 mm, vias 5 -> 1
- net 5V: track 15.8 -> 31.9 mm, vias 2 -> 0
- net N$6: track 0.00 -> 15.7 mm
- net VBAT: track 56.5 -> 71.7 mm
- net BAT+: track 59.3 -> 46.0 mm, vias 5 -> 0
- net N$7: track 0.00 -> 10.9 mm, vias 0 -> 2
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Other:
- board size 144.8 x 55.5 mm -> 142.2 x 47.9 mm

Commit message: updated files even more
Parts:
- moved U$6 44.5 mm to (97.8, 8.89)
- moved U$7 44.5 mm to (97.8, 53.3)
- moved GT_U7_NEO_6M 22.5 mm to (74.9, 26.7)
- moved R2 6.35 mm to (62.2, 49.5), turned to 270 degrees
- moved R1 5.08 mm to (55.9, 49.5), turned to 270 degrees
- moved U$3 5.08 mm to (59.7, 34.3)
- moved C1 4.02 mm to (53.3, 30.5)
- moved C3 4.02 mm to (41.9, 39.4)
- moved R4 3.81 mm to (62.2, 44.5)
- moved U$2 3.81 mm to (48.3, 34.3)
- moved U1 2.84 mm to (34.3, 35.6)
- moved C5 2.54 mm to (30.5, 44.5)
- moved U$8 2.54 mm to (41.9, 35.6)
- moved U$9 2.54 mm to (36.8, 44.5), turned to 90 degrees
- moved U$10 1.80 mm to (55.9, 39.4)
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Routing:
- net GND: track 198.5 -> 0.00 mm, vias 10 -> 0
- net TX2: track 74.1 -> 49.9 mm
- net RX2: track 77.7 -> 54.8 mm
- net SCL: track 43.3 -> 63.8 mm, vias 2 -> 3
- net 3.3V: track 187.5 -> 169.9 mm, vias 4 -> 0
- net MOSI: track 117.5 -> 102.6 mm
- net MISO: track 93.6 -> 83.0 mm, vias 4 -> 6
- net CS3: track 17.2 -> 27.5 mm
- net SCK: track 81.9 -> 71.7 mm
- net N$2: track 26.8 -> 16.7 mm
- net ICMINT1: track 29.7 -> 20.6 mm, vias 0 -> 2
- net SDA: track 47.9 -> 56.4 mm, vias 1 -> 0
- net CS1: track 46.5 -> 38.1 mm
- net CS4: track 34.6 -> 29.1 mm
- net CSN: track 48.7 -> 43.2 mm, vias 0 -> 4
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- removed copper zone on layer 16, net GND
Other:
- board size 142.2 x 47.9 mm -> 99 x 49.2 mm
- board text added: "CSULB Beach Launch Team PCB V2.0"
- board text removed: "AVIONICS BOARD V2.0"
- board text removed: "CSULB BEACH LAUNCH TEAM"

Commit message: Updated files
Routing:
- net CE: track 46.6 -> 47.2 mm
Changed lines of the file:
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@@
 <wire x1="30.48" y1="35.052" x2="30.49" y2="34.925" width="0.1524" layer="1"/>
 <wire x1="28.0416" y1="47.6504" x2="28.0416" y2="53.34" width="0.1524" layer="16"/>
-<wire x1="28.0416" y1="43.18" x2="28.0416" y2="47.6504" width="0.1524" layer="1"/>
-<wire x1="29.718" y1="36.7284" x2="29.4132" y2="37.0332" width="0.1524" layer="1"/>
+<wire x1="28.0416" y1="38.4048" x2="28.0416" y2="47.6504" width="0.1524" layer="1"/>
+<wire x1="29.718" y1="36.7284" x2="28.0416" y2="38.4048" width="0.1524" layer="1"/>
 <wire x1="28.0416" y1="53.34" x2="27.94" y2="53.34" width="0.1524" layer="16"/>
 <via x="52.578" y="34.29" extent="1-16" drill="0.35"/>
@@
 <wire x1="45.72" y1="27.7368" x2="46.3042" y2="28.321" width="0.1524" layer="16"/>
 <wire x1="46.3042" y1="28.321" x2="47.879" y2="28.321" width="0.1524" layer="16"/>
-<wire x1="29.4132" y1="37.0332" x2="29.4132" y2="41.8084" width="0.1524" layer="1"/>
-<wire x1="29.4132" y1="41.8084" x2="28.0416" y2="43.18" width="0.1524" layer="1"/>
 </signal>
 <signal name="MISO">
@@
 <contactref element="U$1" pad="9-OUT1C"/>
 <contactref element="NRF24L01_A" pad="2"/>
+<wire x1="31.6992" y1="11.43" x2="31.6992" y2="17.78" width="0.1524" layer="16"/>
+<wire x1="27.8892" y1="40.5384" x2="26.7208" y2="41.7068" width="0.1524" layer="16"/>
+<wire x1="26.7208" y1="53.34" x2="26.7208" y2="41.7068" width="0.1524" layer="16"/>
 <wire x1="31.75" y1="11.43" x2="31.6992" y2="11.43" width="0.1524" layer="16"/>
 <wire x1="25.4" y1="53.34" x2="26.7208" y2="53.34" width="0.1524" layer="16"/>
-<wire x1="26.7208" y1="53.34" x2="26.7208" y2="46.99" width="0.1524" layer="16"/>
-<wire x1="27.55275625" y1="40.25275625" x2="27.2768" y2="40.5287125" width="0.1524" layer="16"/>
-<wire x1="27.2768" y1="46.434" x2="26.7208" y2="46.99" width="0.1524" layer="16"/>
-<wire x1="31.6992" y1="11.43" x2="31.6992" y2="20.3708" width="0.1524" layer="16"/>
-<wire x1="31.6992" y1="20.3708" x2="27.7761" y2="24.2939" width="0.1524" layer="16"/>
-<wire x1="27.2768" y1="40.5287125" x2="27.2768" y2="46.434" width="0.1524" layer="16"/>
-<wire x1="28.80299375" y1="27.6526" x2="28.9226" y2="27.6526" width="0.1524" layer="16"/>
-<wire x1="28.9226" y1="27.6526" x2="29.21" y2="27.94" width="0.1524" layer="16"/>
-<wire x1="27.7761" y1="24.2939" x2="27.7761" y2="26.62570625" width="0.1524" layer="16"/>
-<wire x1="27.7761" y1="26.62570625" x2="28.80299375" y2="27.6526" width="0.1524" layer="16"/>
-<wire x1="27.7761" y1="40.0294125" x2="27.55275625" y2="40.25275625" width="0.1524" layer="16"/>
-<wire x1="27.7761" y1="38.2639" x2="27.7761" y2="40.0294125" width="0.1524" layer="16"/>
-<wire x1="29.21" y1="27.94" x2="29.21" y2="36.83" width="0.1524" layer="16"/>
-<wire x1="29.21" y1="36.83" x2="27.7761" y2="38.2639" width="0.1524" layer="16"/>
+<wire x1="31.6992" y1="17.78" x2="27.8892" y2="21.59" width="0.1524" layer="16"/>
+<wire x1="27.8892" y1="21.59" x2="27.8892" y2="27.94" width="0.1524" layer="16"/>
+<wire x1="27.8892" y1="27.94" x2="27.8892" y2="40.5384" width="0.1524" layer="16"/>
+<wire x1="27.8892" y1="27.94" x2="27.8892" y2="27.94" width="0.1524" layer="16"/>
+<wire x1="27.8892" y1="27.94" x2="29.1592" y2="29.21" width="0.1524" layer="16"/>
+<wire x1="29.1592" y1="29.21" x2="29.21" y2="29.21" width="0.1524" layer="16"/>
 </signal>
 <signal name="CSN">

Commit message: updated files
Parts:
- removed GT_U7_NEO_6M: (no value), SparkFun-Connectors:1X05
- moved C6 1.80 mm to (40.6, 50.8)
Connections:
- net 3.3V: no longer GT_U7_NEO_6M.5
- net GND: no longer GT_U7_NEO_6M.4
- net RX2: no longer GT_U7_NEO_6M.2
- net TX2: no longer GT_U7_NEO_6M.3
Routing:
- net 3.3V: track 169.9 -> 0.00 mm
- net MOSI: track 102.6 -> 0.00 mm, vias 2 -> 0
- net MISO: track 83.0 -> 0.00 mm, vias 6 -> 0
- net VBAT: track 72.1 -> 0.00 mm
- net SCK: track 71.7 -> 0.00 mm, vias 2 -> 0
- net SCL: track 63.8 -> 0.00 mm, vias 3 -> 0
- net BMPINT: track 60.3 -> 0.00 mm
- net SDA: track 56.4 -> 0.00 mm
- net RX2: track 54.8 -> 0.00 mm
- net TX2: track 49.9 -> 0.00 mm
- net CE: track 47.2 -> 0.00 mm
- net BAT+: track 45.5 -> 0.00 mm, vias 1 -> 0
- net CSN: track 43.2 -> 0.00 mm, vias 4 -> 0
- net CS1: track 38.1 -> 0.00 mm
- net 5V: track 32.0 -> 0.00 mm
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
Commit message: Updated files
Parts:
- removed 3.3V_BUCK_CONVERTER, 5V_BUCK_CONVERTER: (no value), SparkFun-Connectors:1X04
- added C10, C11, C7, C8, C9: 0.1uF, SparkFun-Capacitors:0603
- added U$11: BUCK_CONVERTER5V, BLTFootprints:1X04
- added U$12: BUCK_CONVERTER3.3V, BLTFootprints:1X04
- moved C5 19.7 mm to (49.5, 49.5)
- moved C4 14.5 mm to (44.5, 52.1)
- moved R2 12.0 mm to (50.8, 45.7)
- moved Y1 10.2 mm to (45.7, 49.5)
- moved U$8 7.18 mm to (47.0, 40.6)
- moved R3 5.24 mm to (50.8, 43.2)
- moved U$9 5.08 mm to (41.9, 44.5)
- moved C1 3.81 mm to (49.5, 30.5)
- moved C3 2.84 mm to (44.5, 40.6)
- moved C2 2.84 mm to (49.5, 36.8)
- moved U$3 2.54 mm to (57.1, 34.3)
- moved C6 1.27 mm to (39.4, 50.8)
Connections:
- net 3.3V: now also C10.1, C11.1, C7.1, C8.1, C9.1, U$12.IN+; no longer 3.3V_BUCK_CONVERTER.4
- net 5V: now also U$11.IN+; no longer 5V_BUCK_CONVERTER.4
- net BAT+: now also U$11.VO+, U$12.VO+; no longer 3.3V_BUCK_CONVERTER.2, 5V_BUCK_CONVERTER.2
- net GND: now also C10.2, C11.2, C7.2, C8.2, C9.2, U$11.GND, U$12.GND; no longer 3.3V_BUCK_CONVERTER.3, 5V_BUCK_CONVERTER.3
