File: BLT_Preliminary_Avionics_Schematic_Brandon_update_August_8_2021.sch (EAGLE design)
At the start: 27 parts, among them Y1 32.768kHz

Commit message: updated files
Parts:
- removed GT_U7_NEO_6M: (no value), SparkFun-Connectors:CONN_05
Connections:
- net 3.3V: no longer GT_U7_NEO_6M.5
- net GND: no longer GT_U7_NEO_6M.4
- net RX2: no longer GT_U7_NEO_6M.2
- net TX2: no longer GT_U7_NEO_6M.3
Changed lines of the file:
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@@
 <drawing>
 <settings>
-<setting alwaysvectorfont="no"/>
+<setting alwaysvectorfont="yes"/>
 <setting verticaltext="up"/>
 </settings>
@@
 <part name="3.3V_BUCK_CONVERTER" library="SparkFun-Connectors" deviceset="CONN_04" device="PTH"/>
 <part name="2_CELL_LIPO_BATTERY" library="SparkFun-Connectors" deviceset="CONN_02" device=""/>
-<part name="GT_U7_NEO_6M" library="SparkFun-Connectors" deviceset="CONN_05" device=""/>
 <part name="BT1" library="Battery_Holder" library_urn="urn:adsk.eagle:library:27510219" deviceset="COIN-CELL-THM-3P?-" device="-3003" package3d_urn="urn:adsk.eagle:package:27510259/2" technology="CR2032" value="CR2032"/>
 <part name="U1" library="Adafruit SPI Flash SD Card" deviceset="MICROBUILDER_SMT_SDCARD_8PIN" device=""/>
@@
 <attribute name="NAME" x="35.56" y="102.108" size="1.778" layer="95" font="vector"/>
 </instance>
-<instance part="GT_U7_NEO_6M" gate="G$1" x="127" y="25.4" smashed="yes" rot="R180">
-<attribute name="VALUE" x="129.54" y="35.306" size="1.778" layer="96" font="vector" rot="R180"/>
-<attribute name="NAME" x="132.08" y="17.272" size="1.778" layer="95" font="vector" rot="R180"/>
-</instance>
 <instance part="BT1" gate="G$1" x="162.56" y="45.72" smashed="yes">
 <attribute name="NAME" x="161.29" y="52.07" size="1.778" layer="95" align="center"/>
@@
 <wire x1="119.38" y1="104.14" x2="114.3" y2="104.14" width="0.1524" layer="91"/>
 <label x="111.76" y="104.14" size="1.778" layer="95"/>
-</segment>
-<segment>
-<pinref part="GT_U7_NEO_6M" gate="G$1" pin="5"/>
-<wire x1="119.38" y1="20.32" x2="114.3" y2="20.32" width="0.1524" layer="91"/>
-<label x="111.76" y="20.32" size="1.778" layer="95"/>
 </segment>
 <segment>
@@
 </segment>
 <segment>
-<pinref part="GT_U7_NEO_6M" gate="G$1" pin="4"/>
-<wire x1="119.38" y1="22.86" x2="114.3" y2="22.86" width="0.1524" layer="91"/>
-<label x="111.76" y="22.86" size="1.778" layer="95"/>
-</segment>
-<segment>
 <pinref part="U$1" gate="G$1" pin="GND1"/>
 <wire x1="43.18" y1="-5.08" x2="43.18" y2="-7.62" width="0.1524" layer="91"/>
@@
 <segment>
 <pinref part="C3" gate="G$1" pin="2"/>
-<wire x1="246.38" y1="142.24" x2="248.92" y2="142.24" width="0.1524" layer="91"/>
-<label x="248.92" y="142.24" size="1.778" layer="95"/>
+<wire x1="246.38" y1="142.24" x2="246.38" y2="139.7" width="0.1524" layer="91"/>
+<label x="246.38" y="139.7" size="1.778" layer="95"/>
 </segment>
 <segment>
@@
 <segment>
 <wire x1="111.76" y1="93.98" x2="111.76" y2="88.9" width="0.1524" layer="91"/>
-<label x="111.76" y="93.98" size="1.778" layer="95"/>
+<label x="104.14" y="91.44" size="1.778" layer="95"/>
 <pinref part="NRF24L01_A" gate="G$1" pin="1"/>
 <wire x1="111.76" y1="76.2" x2="111.76" y2="86.36" width="0.1524" layer="91"/>
@@
 <wire x1="111.76" y1="88.9" x2="119.38" y2="88.9" width="0.1524" layer="91"/>
 <junction x="119.38" y="88.9"/>
+<wire x1="111.76" y1="93.98" x2="109.22" y2="93.98" width="0.1524" layer="91"/>
+<wire x1="109.22" y1="93.98" x2="109.22" y2="91.44" width="0.1524" layer="91"/>
 </segment>
 </net>
@@
 <net name="TX2" class="0">
 <segment>
-<pinref part="GT_U7_NEO_6M" gate="G$1" pin="3"/>
-<wire x1="119.38" y1="25.4" x2="114.3" y2="25.4" width="0.1524" layer="91"/>
-<label x="111.76" y="25.4" size="1.778" layer="95"/>
-</segment>
-<segment>
 <pinref part="U$1" gate="G$1" pin="8-TX2/IN1"/>
 <wire x1="78.74" y1="50.8" x2="86.36" y2="50.8" width="0.1524" layer="91"/>
@@
 <net name="RX2" class="0">
 <segment>
-<pinref part="GT_U7_NEO_6M" gate="G$1" pin="2"/>
-<wire x1="119.38" y1="27.94" x2="114.3" y2="27.94" width="0.1524" layer="91"/>
-<label x="111.76" y="27.94" size="1.778" layer="95"/>
-</segment>
-<segment>
 <pinref part="U$1" gate="G$1" pin="7-RX2/OUT1A"/>

Commit message: Updated files
Parts:
- removed 3.3V_BUCK_CONVERTER, 5V_BUCK_CONVERTER: (no value), SparkFun-Connectors:CONN_04PTH
- added C10, C11, C7, C8, C9: 0.1uF, SparkFun-Capacitors:0.1UF-0603-100V-10%
- added U$11: BUCK_CONVERTER5V, BLTFootprints:BUCK_CONVERTER5V
- added U$12: BUCK_CONVERTER3.3V, BLTFootprints:BUCK_CONVERTER3.3V
Connections:
- net 3.3V: now also C10.1, C11.1, C7.1, C8.1, C9.1, U$12.IN+; no longer 3.3V_BUCK_CONVERTER.4
- net 5V: now also U$11.IN+; no longer 5V_BUCK_CONVERTER.4
- net BAT+: now also U$11.VO+, U$12.VO+; no longer 3.3V_BUCK_CONVERTER.2, 5V_BUCK_CONVERTER.2
- net GND: now also C10.2, C11.2, C7.2, C8.2, C9.2, U$11.GND, U$12.GND; no longer 3.3V_BUCK_CONVERTER.3, 5V_BUCK_CONVERTER.3
Other:
- moved on the sheet: BT1, C1, U$2, U$3, U1
