File: Teensy 3.2 reference board clone/T32 ref.brd (EAGLE design)
At the start: 160 x 100 mm, 75 parts, among them K1 MK20DX256VLH7, K2 MKL04Z32VLC4, T1 MCP1825S, U3 SN65HVD230, U4 W25Q32FV, U6 MAX17632AATE+T21-0136I_T1633-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, Y1 32.768kHz, Y2 32.768kHz, Y3 16MHZ

Commit message: /
Parts:
- removed J1: (no value), SparkFun-Connectors:USB-B-MICRO-SMD
- removed K2: MKL04Z32VLC4, t32_ref:LQFP32-08
- removed PROGSW: (no value), SparkFun-Connectors:1X02
- removed SJ1: (no value), t32_ref:SOLDERJUMPER
- removed SX2, SX38, SX40, SX57, SX58, SX59: PIN, t32_ref:PTH_39MIL
- removed T1: MCP1825S, t32_ref:SOT-223
- added C31: 2.2uF, SparkFun-Capacitors:0603
- added J2: 1-2295018-2, 1-2295018-2:TE_1-2295018-2
- added J3: (no value), SparkFun-Connectors:1X07
- added R14, R15: 1.5K, OPL_Resistor:R0603
- added U1: LP38691QSD-3.3/NOPBSDE06A_TEX-M, BLTFootprints:SDE06A_TEX-M
- added U5: MKL02Z32VFG4, MKL02Z32VFG4:QFN50P300X300X65-17N
- C1: device t32_ref:C0603 -> SparkFun-Capacitors:0603
- moved K1 89.6 mm to (40.6, 39.4)
- moved U$2 85.2 mm to (38.1, 66.0)
- moved U$10 75.6 mm to (34.3, 61.0)
- moved R13 74.1 mm to (48.3, 29.2)
- moved U3 73.7 mm to (43.2, 24.1)
- moved U$3 71.4 mm to (14.0, 73.7)
- moved C2 54.3 mm to (-6.35, 49.5)
- moved NRF24L01_B 53.9 mm to (11.4, 62.2)
- moved C1 49.6 mm to (-64.8, 57.1)
- moved C15 44.5 mm to (-19.1, 61.0)
- moved R1 42.0 mm to (-15.2, 43.2)
- moved R11 42.0 mm to (-15.2, 57.1)
- moved R12 42.0 mm to (-20.3, 57.1)
- moved R10 41.9 mm to (-19.1, 64.8)
- moved R9 41.9 mm to (-15.2, 64.8)
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Connections:
- net N$1 renamed XTAL32
- net N$11 renamed VREF_OUT
- net N$13 renamed AREF+
- net N$2 renamed EXTAL32
- net N$20 renamed BNO_XIN32
- net N$21 renamed A9
- net N$22 renamed A8
- net N$23 renamed A7
- net N$24 renamed A6
- net N$27 renamed A3
- net N$28 renamed A2
- net N$29 renamed A1
- net N$30 renamed A0
- net N$39 renamed MCU_5
- net N$42 renamed MCU_2
- net N$43 renamed MCU_1
- net N$44 renamed MCU_0
- net N$45 renamed A13
- net N$46 renamed MCU_33
- net N$47 renamed MCU_32
- net N$48 renamed MCU_31
- net N$49 renamed MCU_30
- net N$5 renamed PTA19
- net N$50 renamed MCU_29
- net N$51 renamed MCU_28
- net N$54 renamed A14
- net N$55 renamed A12
- net N$56 renamed BNO_XOUT32
- net N$57 renamed MCU_24
- net N$58 renamed MCU_25
- net N$59 renamed MCU_26
- net N$60 renamed MCU_27
- net N$64 renamed A11+
- net N$65 renamed A10+
- net N$68 renamed MCU_BATIN
- net N$7 renamed PTA18
- net N$71 renamed BNO_SDA_OUT
- net N$72 renamed BNO_SCL_OUT
- removed net N$15: C6.1, K1.13, R2.1, R3.1
- removed net N$16: J1.D+, R6.1
- removed net N$17: J1.D-, R5.1
- removed net N$19: J1.ID, K1.23, K2.10
- removed net N$3: K1.24, K2.17
- new net EXP: U5.17
- new net N$1: J2.A5, R14.2
- new net N$2: J2.B5, R15.1
- new net PTA2: K1.24, U5.9
- new net USB_D+: J2.A6, J2.B7, R6.1
- new net USB_D-: J2.A7, J2.B6, R5.1
- new net USB_ID: K1.23, U5.6
- new net VDDA: C6.1, K1.13, R2.2, R3.1
- net 3.3V: now also J3.1, R2.1, U1.4, U1.5, U5.1; no longer K2.3, K2.4, R2.2, T1.3
- net 5V: now also C31.1, U1.1, U1.6; no longer SJ1.1, SJ1.2, SX2.1, T1.1
- net EN': now also J3.4, U5.3; no longer K2.7, SX59.1
- net GND: now also C31.2, J2.A1, J2.A12, J2.B1, J2.B12, J2.S1, J2.S2, J2.S3, J2.S4, J3.2, R14.1, R15.2, U1.2, U5.2; no longer J1.GND, J1.SHIELD1, J1.SHIELD2, J1.SHIELD3, K2.5, K2.6, PROGSW.2, T1.2, T1.PAD
- net PROG: now also J3.3, U5.10; no longer K2.18, PROGSW.1, SX40.1
- net RESET: now also J3.7, U5.4, U5.5; no longer K2.25, K2.8, SX38.1
- net SWC: now also J3.5, U5.8; no longer K2.16, SX58.1
- net SWD: now also J3.6, U5.7; no longer K2.15, SX57.1
- net VUSB: now also J2.A4, J2.A9, J2.B4, J2.B9; no longer J1.VBUS
