File: Teensy 3.2 reference board clone/T32 ref.sch (EAGLE design)
At the start: 70 parts, among them K1 MK20DX256VLH7, K2 MKL04Z32VLC4, T1 MCP1825S, U3 SN65HVD230, U4 W25Q32FV, X1 MINI-USB, Y1 32.768kHz

Commit message: Updated files
Parts:
- removed G1: 16MHz, t32_ref:CRYSTAL-HC49US
- removed G2: 32.768kHz, t32_ref:CRYSTAL-TC26H
- removed S1: (no value), t32_ref:TACT_SWITCH
- removed SX3: PIN, t32_ref:PIN
- added PROGSW: (no value), SparkFun-Connectors:CONN_02
- added Y2: 32.768kHz, SparkFun-Clocks:CRYSTAL-32.768KHZSMD-3.2X1.5
- added Y3: 16MHZ, OPL_Crystal Oscillator:SMD-CRYSTAL-16MHZ-8PF-20PPM-40R(2P-5.0X3.2MM)
Connections:
- removed net N$6: C11.1, G1.2, K1.PTA19
- removed net N$8: G2.2, K1.EXTAL32
- new net N$1: K1.XTAL32, Y2.2
- new net N$2: K1.EXTAL32, Y2.1
- net AGND: no longer SX3.P$1
- net GND: now also PROGSW.2; no longer S1.3
- net N$5: now also C11.1, K1.PTA19, Y3.1; no longer C10.1, G1.1, K1.PTA18
- net N$7: now also C10.1, K1.PTA18, Y3.2; no longer G2.1, K1.XTAL32
- net PROG: now also PROGSW.1; no longer S1.1
Other:
- note removed: "GND"
- note removed: "VBAT"

Commit message: /
Parts:
- removed K2: MKL04Z32VLC4, t32_ref:MKL04Z32VLC4
- removed PROGSW: (no value), SparkFun-Connectors:CONN_02
- removed SJ1: (no value), t32_ref:SOLDERJUMPER
- removed SX2, SX38, SX40, SX57, SX58, SX59: PIN, t32_ref:PIN
- removed T1: MCP1825S, t32_ref:LDO
- removed U$12: BUCK_CONVERTER3.3V, BLTFootprints:BUCK_CONVERTER3.3V
- removed X1: MINI-USB, t32_ref:MINI-USBMOLEX_0675031230
- added C26: 0.1uF, SparkFun-Capacitors:0.1UF-0603-25V-(+80/-20%)
- added C27, C28: 22UF-1210-16V-20%, SparkFun-Capacitors:22UF-1210-16V-20%
- added C29, C30, C31: 2.2uF, SparkFun-Capacitors:2.2UF-0603-10V-20%
- added J2: 1-2295018-2, 1-2295018-2:1-2295018-2
- added J3: (no value), SparkFun-Connectors:CONN_07
- added L1: MLF1608E6R8KTD25, MLF1608E6R8KTD25:MLF1608E6R8KTD25
- added R14, R15: 1.5K, OPL_Resistor:SMD-RES-5.1K-1%-1/10W(0603)
- added SPI_SD_CARD: (no value), Adafruit SPI Flash SD Card:MICROBUILDER_SMT_SDCARD_8PIN
- added U5: MKL02Z32VFG4, MKL02Z32VFG4:MKL02Z32VFG4
- added U6: MAX17632AATE+T21-0136I_T1633-5_MXM-M, BLTFootprints:MAX17632AATE+T21-0136I_T1633-5_MXM-M
- C1: device t32_ref:CAPACITOR-0.1UF -> SparkFun-Capacitors:0.1UF-0603-25V-(+80/-20%)
- C2: device t32_ref:CAPACITOR-2.2UF -> SparkFun-Capacitors:2.2UF-0603-10V-20%
- U1: value (none) -> LP38691QSD-3.3/NOPBSDE06A_TEX-M; device Adafruit SPI Flash SD Card:MICROBUILDER_SMT_SDCARD_8PIN -> BLTFootprints:LP38691QSD-3.3/NOPBSDE06A_TEX-M
Connections:
- net N$1 renamed XTAL32
- net N$11 renamed VREF_OUT
- net N$13 renamed AREF+
- net N$2 renamed EXTAL32
- net N$20 renamed BNO_XIN32
- net N$21 renamed A9
- net N$22 renamed A8
- net N$23 renamed A7
- net N$24 renamed A6
- net N$27 renamed A3
- net N$28 renamed A2
- net N$29 renamed A1
- net N$30 renamed A0
- net N$39 renamed MCU_5
- net N$42 renamed MCU_2
- net N$43 renamed MCU_1
- net N$44 renamed MCU_0
- net N$45 renamed A13
- net N$46 renamed MCU_33
- net N$47 renamed MCU_32
- net N$48 renamed MCU_31
- net N$49 renamed MCU_30
- net N$5 renamed PTA19
- net N$50 renamed MCU_29
- net N$51 renamed MCU_28
- net N$54 renamed A14
- net N$55 renamed A12
- net N$56 renamed BNO_XOUT32
- net N$57 renamed MCU_24
- net N$58 renamed MCU_25
- net N$59 renamed MCU_26
- net N$60 renamed MCU_27
- net N$64 renamed A11+
- net N$65 renamed A10+
- net N$68 renamed MCU_BATIN
- net N$7 renamed PTA18
- net N$71 renamed BNO_SDA_OUT
- net N$72 renamed BNO_SCL_OUT
- removed net N$15: C6.1, K1.VDDA, R2.1, R3.1
- removed net N$16: R6.1, X1.3
- removed net N$17: R5.1, X1.2
- removed net N$19: K1.PTA1, K2.PTA6, X1.4
- removed net N$3: K1.PTA2, K2.PTB1
- new net BUCK_3.3V_BST: C26.1, U6.BST
- new net BUCK_3.3V_LX: C26.2, L1.1, U6.LX, U6.LX_2
- new net BUCK_3.3V_VCC: C29.1
- new net N$1: J2.CC1, R14.2
- new net N$2: J2.CC2, R15.1
- new net PTA2: K1.PTA2, U5.PTB1/IRQ_6
- new net USB_D+: J2.D+_A, J2.D-_B, R6.1
- new net USB_D-: J2.D+_B, J2.D-_A, R5.1
- new net USB_ID: K1.PTA1, U5.PTA6
- new net VDDA: C6.1, K1.VDDA, R2.2, R3.1
- net 3.3V: now also C27.1, C28.1, J3.1, L1.2, R2.1, SPI_SD_CARD.VCC, U1.SNS, U1.VOUT, U5.VDD/VREFH, U6.FB; no longer K2.VDD, K2.VREFH, R2.2, T1.OUT, U$12.IN+, U1.VCC
- net 5V: now also C31.1, U1.VIN, U1.VIN_2; no longer SJ1.1, SJ1.2, SX2.P$1, T1.IN
- net BAT+: now also C30.1, U6.EN/UVLO, U6.VCC, U6.VIN, U6.VIN_2; no longer U$12.VO+
- net CS1: now also SPI_SD_CARD.SSEL/SD3; no longer U1.SSEL/SD3
- net EN': now also J3.4, U5.PTA3; no longer K2.PTA3, SX59.P$1
- net GND: now also C27.2, C28.2, C29.2, C30.2, C31.2, J2.GND_A, J2.GND_B, J2.SHIELD, J3.2, R14.1, R15.2, SPI_SD_CARD.VSS, U1.GND, U5.VREFL/VSS, U6.EXTVCC, U6.MODE/SYNC, U6.PGND, U6.PGND_2, U6.SGND; no longer K2.VREFL, K2.VSS, PROGSW.2, T1.GND, T1.PAD, U$12.GND, U1.VSS, X1.5, X1.CASE
- net MISO: now also SPI_SD_CARD.MISO/SD0; no longer U1.MISO/SD0
- net MOSI: now also SPI_SD_CARD.MOSI/CMD; no longer U1.MOSI/CMD
- net PROG: now also J3.3, U5.PTB2/IRQ_7; no longer K2.PTB2, PROGSW.1, SX40.P$1
- net RESET: now also J3.7, U5.PTA4, U5.PTA5; no longer K2.PTA4, K2.PTB5, SX38.P$1
- net SCK: now also SPI_SD_CARD.SCK; no longer U1.SCK
- net SWC: now also J3.5, U5.PTB0/IRQ_5; no longer K2.PTB0, SX58.P$1
- net SWD: now also J3.6, U5.PTA7/IRQ_4; no longer K2.PTA7, SX57.P$1
- net VUSB: now also J2.VBUS_A, J2.VBUS_B; no longer X1.1
Other:
- note removed: "0"
- note removed: "1"
- note removed: "14 / A0"
- note removed: "15 / A1"
- note removed: "16 / A2"
- note removed: "17 / A3"
- note removed: "2"
- note removed: "20 / A6"
- note removed: "21 / A7"
- note removed: "22 / A8"
- note removed: "23 / A9"
- note removed: "24"
- note removed: "25"
- note removed: "26"
- note removed: "27"
- note removed: "28"
- note removed: "29"
- note removed: "3"
- note removed: "30"
- note removed: "31"
- note removed: "32"
- note removed: "33"
- note removed: "4"
- note removed: "5"
- note removed: "6"
- note removed: "7"
- note removed: "8"
- note removed: "9"
- note removed: "A10"
- note removed: "A11"
- note removed: "A12"
- note removed: "A13"
- note removed: "AGND"
- note removed: "AREF"
- note removed: "DAC / A14"
- note removed: "EN'"
- note removed: "PROG"
- note removed: "RESET"
- note removed: "SWC"
- note removed: "SWD"
- note removed: "VIN"
- moved on the sheet: 2_CELL_LIPO_BATTERY, C10, C11, C12, C18, C24, C3, C4, C5, C6, C7, C8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
